Commit message: gazebo 可以正常运行

File: all_wheel_description/urdf/all_wheel.urdf (robot description, URDF)
Before this commit: robot ALL_WHEEL, 5 links, 4 joints
Links:
- added link base_footprint
- link base_link: geometry collision mesh filename=file:///home/shexingju/code/ROS/ALL_WHEEL_CHASSIS/install/a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; visual mesh filename=file:///home/shexingju/code/ROS/ALL_WHEEL_CHASSIS/install/a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
- link front_link: geometry collision mesh filename=file:///home/shexingju/code/ROS/ALL_WHEEL_CHASSIS/install/a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; visual mesh filename=file:///home/shexingju/code/ROS/ALL_WHEEL_CHASSIS/install/a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
- link imu_Link: mass 0.025372414405334 -> 0.0283869958164694; geometry collision mesh filename=file:///home/shexingju/code/ROS/ALL_WHEEL_CHASSIS/install/a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; visual mesh filename=file:///home/shexingju/code/ROS/ALL_WHEEL_CHASSIS/install/a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
- link left_Link: geometry collision mesh filename=file:///home/shexingju/code/ROS/ALL_WHEEL_CHASSIS/install/a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; visual mesh filename=file:///home/shexingju/code/ROS/ALL_WHEEL_CHASSIS/install/a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
- link right_Link: geometry collision mesh filename=file:///home/shexingju/code/ROS/ALL_WHEEL_CHASSIS/install/a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; visual mesh filename=file:///home/shexingju/code/ROS/ALL_WHEEL_CHASSIS/install/a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
Joints:
- added joint base_footprint_to_base_link: type fixed, parent base_footprint, child base_link, origin xyz=0 0 0 rpy=0 0 0

Commit message: 支持相对路径

File: all_wheel_description/urdf/all_wheel.urdf (robot description, URDF)
Before this commit: robot allwheel_urdf, 6 links, 5 joints
Links:
- link base_link: geometry collision mesh filename=package://all_wheel_description/meshes/base_link.STL; visual mesh filename=package://all_wheel_description/meshes/base_link.STL
- link front_link: geometry collision mesh filename=package://all_wheel_description/meshes/front_link.STL; visual mesh filename=package://all_wheel_description/meshes/front_link.STL
- link imu_Link: geometry collision mesh filename=package://all_wheel_description/meshes/imu_Link.STL; visual mesh filename=package://all_wheel_description/meshes/imu_Link.STL
- link left_Link: geometry collision mesh filename=package://all_wheel_description/meshes/left_Link.STL; visual mesh filename=package://all_wheel_description/meshes/left_Link.STL
- link right_Link: geometry collision mesh filename=package://all_wheel_description/meshes/right_Link.STL; visual mesh filename=package://all_wheel_description/meshes/right_Link.STL

Commit message: 支持双目相机

File: all_wheel_description/urdf/all_wheel.urdf (robot description, URDF)
Before this commit: robot allwheel_urdf, 6 links, 5 joints
Links:
- added link left_camera_link, mass 0.02
- added link right_camera_link, mass 0.02
Joints:
- added joint left_camera_joint: type fixed, parent base_link, child left_camera_link, origin xyz=0.12 0.05 0.10 rpy=0 0 0
- added joint right_camera_joint: type fixed, parent base_link, child right_camera_link, origin xyz=0.12 -0.05 0.10 rpy=0 0 0

Commit message: 增加激光雷达

File: all_wheel_description/urdf/all_wheel.urdf (robot description, URDF)
Before this commit: robot allwheel_urdf, 8 links, 7 joints
Links:
- added link lidar_link, mass 0.05
Joints:
- added joint lidar_joint: type fixed, parent base_link, child lidar_link, origin xyz=0.12 0 0.12 rpy=0 0 0
